File: Commodore/2031/2031040/Commodore-2031/Sheet1-ReadWriteLogic.kicad_sch (KiCad schematic)
At the start: 14 parts

Commit message: Capture sheet 3
Connections:
- net GND: now also UL5.1 (P1), UL5.10 (P2), UL5.15 (P0), UL5.4 (Ce), UL5.5 (D/U)
- net at UK2.8 (CP), UL3.2 (CP), UL6.9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: now also UK6.1, UL5.14 (Cp), UN2.2 (QB)
Changed lines of the file:
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@@
     (comment 2 "PCB Assembly 2031040")
   )
-  (junction (at 148.59 208.28) (diameter 0) (color 0 0 0 0)
+  (junction (at 143.51 208.28) (diameter 0) (color 0 0 0 0)
+  )
+  (junction (at 264.16 93.98) (diameter 0) (color 0 0 0 0)
+  )
+  (junction (at 328.93 196.85) (diameter 0) (color 0 0 0 0)
   )
   (junction (at 198.12 110.49) (diameter 0) (color 0 0 0 0)
@@
   (junction (at 269.24 142.24) (diameter 0) (color 0 0 0 0)
   )
-  (junction (at 148.59 218.44) (diameter 0) (color 0 0 0 0)
+  (junction (at 143.51 218.44) (diameter 0) (color 0 0 0 0)
   )
   (junction (at 143.51 143.51) (diameter 0) (color 0 0 0 0)
@@
   (junction (at 304.8 179.07) (diameter 0) (color 0 0 0 0)
   )
-  (junction (at 148.59 205.74) (diameter 0) (color 0 0 0 0)
+  (junction (at 143.51 205.74) (diameter 0) (color 0 0 0 0)
   )
   (junction (at 266.7 207.01) (diameter 0) (color 0 0 0 0)
@@
   )
   (junction (at 200.66 93.98) (diameter 0) (color 0 0 0 0)
+  )
+  (junction (at 143.51 223.52) (diameter 0) (color 0 0 0 0)
   )
   (junction (at 184.15 93.98) (diameter 0) (color 0 0 0 0)
@@
     (stroke (width 0) (type default))
   )
-  (wire (pts (xy 325.12 247.65) (xy 217.17 247.65))
+  (wire (pts (xy 328.93 247.65) (xy 217.17 247.65))
+    (stroke (width 0) (type default))
+  )
+  (wire (pts (xy 143.51 223.52) (xy 143.51 224.79))
     (stroke (width 0) (type default))
   )
@@
     (stroke (width 0) (type default))
   )
-  (wire (pts (xy 297.18 196.85) (xy 325.12 196.85))
+  (wire (pts (xy 297.18 196.85) (xy 328.93 196.85))
     (stroke (width 0) (type default))
   )
@@
     (stroke (width 0) (type default))
   )
-  (wire (pts (xy 219.71 240.03) (xy 330.2 240.03))
+  (wire (pts (xy 219.71 240.03) (xy 334.01 240.03))
     (stroke (width 0) (type default))
   )
@@
     (stroke (width 0) (type default))
   )
-  (wire (pts (xy 148.59 205.74) (xy 148.59 208.28))
+  (wire (pts (xy 143.51 205.74) (xy 143.51 208.28))
     (stroke (width 0) (type default))
   )
@@
     (stroke (width 0) (type default))
   )
-  (wire (pts (xy 325.12 196.85) (xy 325.12 247.65))
+  (wire (pts (xy 328.93 196.85) (xy 328.93 247.65))
     (stroke (width 0) (type default))
   )
@@
     (stroke (width 0) (type default))
   )
-  (wire (pts (xy 261.62 104.14) (xy 332.74 104.14))
+  (wire (pts (xy 261.62 104.14) (xy 336.55 104.14))
     (stroke (width 0) (type default))
   )
@@
     (stroke (width 0) (type default))
   )
-  (wire (pts (xy 148.59 208.28) (xy 151.13 208.28))
+  (wire (pts (xy 143.51 208.28) (xy 151.13 208.28))
     (stroke (width 0) (type default))
   )
@@
     (stroke (width 0) (type default))
   )
-  (wire (pts (xy 148.59 218.44) (xy 151.13 218.44))
+  (wire (pts (xy 143.51 218.44) (xy 151.13 218.44))
     (stroke (width 0) (type default))
   )
@@
     (stroke (width 0) (type default))
   )
-  (wire (pts (xy 148.59 203.2) (xy 148.59 205.74))
+  (wire (pts (xy 143.51 203.2) (xy 143.51 205.74))
     (stroke (width 0) (type default))
   )
@@
     (stroke (width 0) (type default))
   )
-  (wire (pts (xy 128.27 91.44) (xy 327.66 91.44))
+  (wire (pts (xy 128.27 91.44) (xy 331.47 91.44))
     (stroke (width 0) (type default))
   )
@@
     (stroke (width 0) (type default))
   )
+  (wire (pts (xy 328.93 93.98) (xy 264.16 93.98))
+    (stroke (width 0) (type default))
+  )
   (wire (pts (xy 55.88 95.25) (xy 55.88 97.79))
     (stroke (width 0) (type default))
@@
     (stroke (width 0) (type default))
   )
-  (wire (pts (xy 247.65 86.36) (xy 332.74 86.36))
+  (wire (pts (xy 247.65 86.36) (xy 336.55 86.36))
     (stroke (width 0) (type default))
   )
@@
     (stroke (width 0) (type default))
   )
-  (wire (pts (xy 297.18 194.31) (xy 330.2 194.31))
+  (wire (pts (xy 297.18 194.31) (xy 334.01 194.31))
     (stroke (width 0) (type default))
   )
@@
     (stroke (width 0) (type default))
   )
+  (wire (pts (xy 328.93 196.85) (xy 328.93 93.98))
+    (stroke (width 0) (type default))
+  )
   (wire (pts (xy 133.35 49.53) (xy 127 49.53))
     (stroke (width 0) (type default))
@@
     (stroke (width 0) (type default))
   )
-  (wire (pts (xy 151.13 205.74) (xy 148.59 205.74))
+  (wire (pts (xy 151.13 205.74) (xy 143.51 205.74))
     (stroke (width 0) (type default))
   )
@@
     (stroke (width 0) (type default))
   )
-  (wire (pts (xy 148.59 223.52) (xy 151.13 223.52))
+  (wire (pts (xy 143.51 223.52) (xy 151.13 223.52))
     (stroke (width 0) (type default))
   )
@@
     (stroke (width 0) (type default))
   )
-  (wire (pts (xy 148.59 208.28) (xy 148.59 218.44))
+  (wire (pts (xy 143.51 208.28) (xy 143.51 218.44))
     (stroke (width 0) (type default))
   )
@@
     (stroke (width 0) (type default))
   )
-  (wire (pts (xy 148.59 203.2) (xy 151.13 203.2))
+  (wire (pts (xy 143.51 203.2) (xy 151.13 203.2))
     (stroke (width 0) (type default))
   )
@@
     (stroke (width 0) (type default))
   )
-  (wire (pts (xy 148.59 218.44) (xy 148.59 223.52))
+  (wire (pts (xy 143.51 218.44) (xy 143.51 223.52))
     (stroke (width 0) (type default))
   )
@@
     (stroke (width 0) (type default))
   )
-  (wire (pts (xy 327.66 91.44) (xy 327.66 201.93))
+  (wire (pts (xy 331.47 91.44) (xy 331.47 201.93))
     (stroke (width 0) (type default))
   )
@@
     (stroke (width 0) (type default))
   )
-  (wire (pts (xy 316.23 179.07) (xy 332.74 179.07))
+  (wire (pts (xy 316.23 179.07) (xy 336.55 179.07))
     (stroke (width 0) (type default))
   )
@@
     (stroke (width 0) (type default))
   )
-  (wire (pts (xy 330.2 194.31) (xy 330.2 240.03))
+  (wire (pts (xy 334.01 194.31) (xy 334.01 240.03))
     (stroke (width 0) (type default))
   )
@@
     (stroke (width 0) (type default))
   )
-  (wire (pts (xy 327.66 201.93) (xy 317.5 201.93))
+  (wire (pts (xy 331.47 201.93) (xy 317.5 201.93))
     (stroke (width 0) (type default))
   )
@@
     (effects (font (size 1.27 1.27)) (justify right bottom))
   )
-  (hierarchical_label "~{MODE}" (shape output) (at 332.74 86.36 0) (fields_autoplaced)
+  (hierarchical_label "~{MODE}" (shape output) (at 336.55 86.36 0) (fields_autoplaced)
     (effects (font (size 1.27 1.27)) (justify left))
   )
@@
     (effects (font (size 1.27 1.27)) (justify left))
   )
-  (hierarchical_label "16MHZ" (shape input) (at 332.74 104.14 0) (fields_autoplaced)
+  (hierarchical_label "16MHZ" (shape input) (at 336.55 104.14 0) (fields_autoplaced)
     (effects (font (size 1.27 1.27)) (justify left))
   )
@@
     (effects (font (size 1.27 1.27)) (justify right))
   )
-  (hierarchical_label "D[0..7]" (shape input) (at 54.61 39.37 180) (fields_autoplaced)
+  (hierarchical_label "D[0..7]" (shape tri_state) (at 54.61 39.37 180) (fields_autoplaced)
     (effects (font (size 1.27 1.27)) (justify right))
   )
@@
     (effects (font (size 1.27 1.27)) (justify left))
   )
-  (hierarchical_label "READ_DATA" (shape input) (at 332.74 179.07 0) (fields_autoplaced)
+  (hierarchical_label "READ_DATA" (shape input) (at 336.55 179.07 0) (fields_autoplaced)
     (effects (font (size 1.27 1.27)) (justify left))
   )
@@
         )
       )
+    )
+  )
+  (symbol (lib_id "power:GND") (at 143.51 224.79 0) (unit 1)
+    (in_bom yes) (on_board yes) (dnp no) (fields_autoplaced)
+    (property "Reference" "#PWR053" (at 143.51 231.14 0)
+      (effects (font (size 1.27 1.27)) hide)
+    )
+    (property "Value" "GND" (at 143.51 229.87 0)
+      (effects (font (size 1.27 1.27)))
+    )
+    (property "Footprint" "" (at 143.51 224.79 0)
+      (effects (font (size 1.27 1.27)) hide)
+    )
+    (property "Datasheet" "" (at 143.51 224.79 0)
+      (effects (font (size 1.27 1.27)) hide)
+    )
+    (pin "1")
+    (instances
+      (project "Commodore-2031"
+        (path "/4559151c-aecb-4a2a-972f-dcb7dcb5a3dc/4c109d40-2790-4a3e-a7c4-2172de51732d"
+          (reference "#PWR053") (unit 1)
+        )
+      )

Commit message: Work towards ERC
- Add power flags
- Try to make sense of ground symbols
Connections:
- net GND renamed Earth
Changed lines of the file:
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@@
     )
   )
-  (symbol (lib_id "power:GND") (at 269.24 147.32 0) (unit 1)
+  (symbol (lib_id "power:Earth") (at 269.24 147.32 0) (unit 1)
     (in_bom yes) (on_board yes) (dnp no) (fields_autoplaced)
     (property "Reference" "#PWR015" (at 269.24 153.67 0)
@@
       (effects (font (size 1.27 1.27)) hide)
     )
-    (property "Datasheet" "" (at 269.24 147.32 0)
+    (property "Datasheet" "~" (at 269.24 147.32 0)
       (effects (font (size 1.27 1.27)) hide)
     )
@@
     )
   )
-  (symbol (lib_id "power:GND") (at 146.05 71.12 0) (unit 1)
+  (symbol (lib_id "power:Earth") (at 146.05 71.12 0) (unit 1)
     (in_bom yes) (on_board yes) (dnp no) (fields_autoplaced)
     (property "Reference" "#PWR04" (at 146.05 77.47 0)
@@
       (effects (font (size 1.27 1.27)) hide)
     )
-    (property "Datasheet" "" (at 146.05 71.12 0)
+    (property "Datasheet" "~" (at 146.05 71.12 0)
       (effects (font (size 1.27 1.27)) hide)
     )
@@
     )
   )
-  (symbol (lib_id "power:GND") (at 143.51 224.79 0) (unit 1)
+  (symbol (lib_id "power:Earth") (at 143.51 224.79 0) (unit 1)
     (in_bom yes) (on_board yes) (dnp no) (fields_autoplaced)
     (property "Reference" "#PWR053" (at 143.51 231.14 0)
@@
       (effects (font (size 1.27 1.27)) hide)
     )
-    (property "Datasheet" "" (at 143.51 224.79 0)
+    (property "Datasheet" "~" (at 143.51 224.79 0)
       (effects (font (size 1.27 1.27)) hide)
     )
@@
     )
   )
-  (symbol (lib_id "power:GND") (at 284.48 151.13 0) (unit 1)
+  (symbol (lib_id "power:Earth") (at 284.48 151.13 0) (unit 1)
     (in_bom yes) (on_board yes) (dnp no) (fields_autoplaced)
     (property "Reference" "#PWR016" (at 284.48 157.48 0)
@@
       (effects (font (size 1.27 1.27)) hide)
     )
-    (property "Datasheet" "" (at 284.48 151.13 0)
+    (property "Datasheet" "~" (at 284.48 151.13 0)
       (effects (font (size 1.27 1.27)) hide)
     )
@@
     )
   )
-  (symbol (lib_id "power:GND") (at 163.83 234.95 0) (unit 1)
+  (symbol (lib_id "power:Earth") (at 163.83 234.95 0) (unit 1)
     (in_bom yes) (on_board yes) (dnp no) (fields_autoplaced)
     (property "Reference" "#PWR012" (at 163.83 241.3 0)
@@
       (effects (font (size 1.27 1.27)) hide)
     )
-    (property "Datasheet" "" (at 163.83 234.95 0)
+    (property "Datasheet" "~" (at 163.83 234.95 0)
       (effects (font (size 1.27 1.27)) hide)
     )
@@
     )
   )
-  (symbol (lib_id "power:GND") (at 146.05 134.62 0) (unit 1)
+  (symbol (lib_id "power:Earth") (at 146.05 134.62 0) (unit 1)
     (in_bom yes) (on_board yes) (dnp no) (fields_autoplaced)
     (property "Reference" "#PWR010" (at 146.05 140.97 0)
@@
       (effects (font (size 1.27 1.27)) hide)
     )
-    (property "Datasheet" "" (at 146.05 134.62 0)
+    (property "Datasheet" "~" (at 146.05 134.62 0)
       (effects (font (size 1.27 1.27)) hide)
     )
@@
     )
   )
-  (symbol (lib_id "power:GND") (at 186.69 72.39 0) (unit 1)
+  (symbol (lib_id "power:Earth") (at 186.69 72.39 0) (unit 1)
     (in_bom yes) (on_board yes) (dnp no) (fields_autoplaced)
     (property "Reference" "#PWR06" (at 186.69 78.74 0)
@@
       (effects (font (size 1.27 1.27)) hide)
     )
-    (property "Datasheet" "" (at 186.69 72.39 0)
+    (property "Datasheet" "~" (at 186.69 72.39 0)
       (effects (font (size 1.27 1.27)) hide)
     )
@@
     )
   )
-  (symbol (lib_id "power:GND") (at 201.93 78.74 0) (unit 1)
+  (symbol (lib_id "power:Earth") (at 201.93 78.74 0) (unit 1)
     (in_bom yes) (on_board yes) (dnp no) (fields_autoplaced)
     (property "Reference" "#PWR07" (at 201.93 85.09 0)
@@
       (effects (font (size 1.27 1.27)) hide)
     )
-    (property "Datasheet" "" (at 201.93 78.74 0)
+    (property "Datasheet" "~" (at 201.93 78.74 0)
       (effects (font (size 1.27 1.27)) hide)
     )
@@
     )
   )
-  (symbol (lib_id "power:GND") (at 284.48 226.06 0) (unit 1)
+  (symbol (lib_id "power:Earth") (at 284.48 226.06 0) (unit 1)
     (in_bom yes) (on_board yes) (dnp no) (fields_autoplaced)
     (property "Reference" "#PWR019" (at 284.48 232.41 0)
@@
       (effects (font (size 1.27 1.27)) hide)
     )
-    (property "Datasheet" "" (at 284.48 226.06 0)
+    (property "Datasheet" "~" (at 284.48 226.06 0)
       (effects (font (size 1.27 1.27)) hide)
     )
@@
     )
   )
-  (symbol (lib_id "power:GND") (at 78.74 109.22 0) (unit 1)
+  (symbol (lib_id "power:Earth") (at 78.74 109.22 0) (unit 1)
     (in_bom yes) (on_board yes) (dnp no) (fields_autoplaced)
     (property "Reference" "#PWR02" (at 78.74 115.57 0)
@@
       (effects (font (size 1.27 1.27)) hide)
     )
-    (property "Datasheet" "" (at 78.74 109.22 0)
-      (effects (font (size 1.27 1.27)) hide)
-    )
+    (property "Datasheet" "~" (at 78.74 109.22 0)
+      (effects (font (size 1.27 1.27)) hide)
+    )

Commit message: Verify schematic against parts list
A few discrepancies appear in original, these are noted in schematic.
Other:
- note added: "U3K is 74LS245 in parts list (equivalent?)"
Changed lines of the file:
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@@
     (stroke (width 0) (type default))
+  )
+  (text "U3K is 74LS245 in parts list\n(equivalent?)" (at 140.97 20.32 0)
+    (effects (font (size 1.27 1.27)) (justify left bottom))
   )
   (text "READ/WRITE LOGIC" (at 175.26 256.54 0)
