File: Commodore/2031/2031040/Commodore-2031/Sheet2-DriveSelectIEEE.kicad_sch (KiCad schematic)
At the start: 51 parts

Commit message: Capture sheet 3
Parts:
- removed C3: 47p, symbol Device:C_Small
- UH3: value ~ -> 6522
- US3: value ~ -> LM555
- renumbered C1 to C53, C56 to C58, C2 to C71
Connections:
- net GND: now also UA1.10 (GND), US1.10 (GND)
Changed lines of the file:
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@@
   (junction (at 88.9 68.58) (diameter 0) (color 0 0 0 0)
   )
-  (junction (at 209.55 119.38) (diameter 0) (color 0 0 0 0)
-  )
   (junction (at 209.55 96.52) (diameter 0) (color 0 0 0 0)
   )
@@
   (junction (at 227.33 101.6) (diameter 0) (color 0 0 0 0)
   )
+  (junction (at 176.53 73.66) (diameter 0) (color 0 0 0 0)
+  )
   (junction (at 71.12 104.14) (diameter 0) (color 0 0 0 0)
   )
@@
   )
   (junction (at 92.71 132.08) (diameter 0) (color 0 0 0 0)
-  )
-  (junction (at 209.55 127) (diameter 0) (color 0 0 0 0)
   )
   (junction (at 218.44 68.58) (diameter 0) (color 0 0 0 0)
@@
     (stroke (width 0) (type default))
   )
+  (wire (pts (xy 176.53 73.66) (xy 172.72 73.66))
+    (stroke (width 0) (type default))
+  )
   (wire (pts (xy 91.44 78.74) (xy 91.44 99.06))
     (stroke (width 0) (type default))
@@
     (stroke (width 0) (type default))
   )
-  (wire (pts (xy 176.53 66.04) (xy 176.53 83.82))
+  (wire (pts (xy 176.53 66.04) (xy 176.53 73.66))
     (stroke (width 0) (type default))
   )
@@
     (stroke (width 0) (type default))
   )
-  (wire (pts (xy 209.55 119.38) (xy 209.55 120.65))
-    (stroke (width 0) (type default))
-  )
   (wire (pts (xy 102.87 68.58) (xy 102.87 69.85))
     (stroke (width 0) (type default))
@@
     (stroke (width 0) (type default))
   )
+  (wire (pts (xy 172.72 73.66) (xy 172.72 76.2))
+    (stroke (width 0) (type default))
+  )
   (wire (pts (xy 218.44 60.96) (xy 247.65 60.96))
     (stroke (width 0) (type default))
@@
     (stroke (width 0) (type default))
   )
-  (wire (pts (xy 209.55 127) (xy 209.55 128.27))
+  (wire (pts (xy 200.66 127) (xy 200.66 128.27))
     (stroke (width 0) (type default))
   )
@@
     (stroke (width 0) (type default))
   )
+  (wire (pts (xy 176.53 73.66) (xy 176.53 83.82))
+    (stroke (width 0) (type default))
+  )
   (wire (pts (xy 38.1 99.06) (xy 43.18 99.06))
     (stroke (width 0) (type default))
@@
     (stroke (width 0) (type default))
   )
-  (wire (pts (xy 189.23 119.38) (xy 209.55 119.38))
-    (stroke (width 0) (type default))
-  )
   (wire (pts (xy 191.77 46.99) (xy 191.77 48.26))
     (stroke (width 0) (type default))
@@
     (stroke (width 0) (type default))
   )
-  (wire (pts (xy 209.55 119.38) (xy 247.65 119.38))
+  (wire (pts (xy 189.23 119.38) (xy 247.65 119.38))
     (stroke (width 0) (type default))
   )
@@
     (effects (font (size 1.27 1.27)) (justify right))
   )
-  (hierarchical_label "D[0..7]" (shape bidirectional) (at 33.02 38.1 180) (fields_autoplaced)
+  (hierarchical_label "D[0..7]" (shape tri_state) (at 33.02 38.1 180) (fields_autoplaced)
     (effects (font (size 1.27 1.27)) (justify right))
   )
@@
     )
   )
-  (symbol (lib_id "power:GND") (at 209.55 128.27 0) (unit 1)
-    (in_bom yes) (on_board yes) (dnp no) (fields_autoplaced)
-    (property "Reference" "#PWR034" (at 209.55 134.62 0)
-      (effects (font (size 1.27 1.27)) hide)
-    )
-    (property "Value" "GND" (at 207.01 130.175 0)
+  (symbol (lib_id "power:GND") (at 200.66 128.27 0) (unit 1)
+    (in_bom yes) (on_board yes) (dnp no) (fields_autoplaced)
+    (property "Reference" "#PWR034" (at 200.66 134.62 0)
+      (effects (font (size 1.27 1.27)) hide)
+    )
+    (property "Value" "GND" (at 198.12 130.175 0)
       (effects (font (size 1.27 1.27)) (justify right))
     )
-    (property "Footprint" "" (at 209.55 128.27 0)
-      (effects (font (size 1.27 1.27)) hide)
-    )
-    (property "Datasheet" "" (at 209.55 128.27 0)
+    (property "Footprint" "" (at 200.66 128.27 0)
+      (effects (font (size 1.27 1.27)) hide)
+    )
+    (property "Datasheet" "" (at 200.66 128.27 0)
       (effects (font (size 1.27 1.27)) hide)
     )
@@
     )
   )
+  (symbol (lib_id "power:GND") (at 172.72 76.2 0) (unit 1)
+    (in_bom yes) (on_board yes) (dnp no) (fields_autoplaced)
+    (property "Reference" "#PWR044" (at 172.72 82.55 0)
+      (effects (font (size 1.27 1.27)) hide)
+    )
+    (property "Value" "GND" (at 172.72 81.28 0)
+      (effects (font (size 1.27 1.27)))
+    )
+    (property "Footprint" "" (at 172.72 76.2 0)
+      (effects (font (size 1.27 1.27)) hide)
+    )
+    (property "Datasheet" "" (at 172.72 76.2 0)
+      (effects (font (size 1.27 1.27)) hide)
+    )
+    (pin "1")
+    (instances
+      (project "Commodore-2031"
+        (path "/4559151c-aecb-4a2a-972f-dcb7dcb5a3dc/882d1050-e467-458c-aabe-cad74417742a"
+          (reference "#PWR044") (unit 1)
+        )
+      )
+    )
+  )
   (symbol (lib_id "Device:FerriteBead_Small") (at 245.11 58.42 90) (unit 1)
     (in_bom yes) (on_board yes) (dnp no)
@@
   (symbol (lib_id "Device:C_Small") (at 200.66 123.19 0) (unit 1)
     (in_bom yes) (on_board yes) (dnp no) (fields_autoplaced)
-    (property "Reference" "C2" (at 203.2 122.5613 0)
+    (property "Reference" "C71" (at 203.2 122.5613 0)
       (effects (font (size 1.27 1.27)) (justify left))
     )
@@
       (project "Commodore-2031"
         (path "/4559151c-aecb-4a2a-972f-dcb7dcb5a3dc/882d1050-e467-458c-aabe-cad74417742a"
-          (reference "C2") (unit 1)
+          (reference "C71") (unit 1)
         )
       )
@@
   (symbol (lib_id "Commodore-2031:LM555") (at 80.01 151.13 0) (unit 1)
     (in_bom yes) (on_board yes) (dnp no)
-    (property "Reference" "US3" (at 80.01 151.13 0)
-      (effects (font (size 1.27 1.27)))
-    )
-    (property "Value" "~" (at 80.01 153.67 0)
+    (property "Reference" "US3" (at 80.01 148.59 0)
+      (effects (font (size 1.27 1.27)))
+    )
+    (property "Value" "LM555" (at 80.01 151.13 0)
       (effects (font (size 1.27 1.27)))
     )
@@
         (path "/4559151c-aecb-4a2a-972f-dcb7dcb5a3dc/882d1050-e467-458c-aabe-cad74417742a"
           (reference "#PWR037") (unit 1)
-        )
-      )
-    )
-  )
-  (symbol (lib_id "Device:C_Small") (at 209.55 123.19 0) (unit 1)
-    (in_bom yes) (on_board yes) (dnp no) (fields_autoplaced)
-    (property "Reference" "C3" (at 212.09 122.5613 0)
-      (effects (font (size 1.27 1.27)) (justify left))
-    )
-    (property "Value" "47p" (at 212.09 125.1013 0)
-      (effects (font (size 1.27 1.27)) (justify left))
-    )
-    (property "Footprint" "" (at 209.55 123.19 0)
-      (effects (font (size 1.27 1.27)) hide)
-    )
-    (property "Datasheet" "~" (at 209.55 123.19 0)
-      (effects (font (size 1.27 1.27)) hide)
-    )
-    (pin "1")
-    (pin "2")
-    (instances
-      (project "Commodore-2031"
-        (path "/4559151c-aecb-4a2a-972f-dcb7dcb5a3dc/882d1050-e467-458c-aabe-cad74417742a"
-          (reference "C3") (unit 1)
         )
       )
@@
   (symbol (lib_id "Device:C_Small") (at 74.93 173.99 0) (unit 1)
     (in_bom yes) (on_board yes) (dnp no) (fields_autoplaced)
-    (property "Reference" "C56" (at 72.39 173.3613 0)
+    (property "Reference" "C58" (at 72.39 173.3613 0)
       (effects (font (size 1.27 1.27)) (justify right))
     )
@@
       (project "Commodore-2031"
         (path "/4559151c-aecb-4a2a-972f-dcb7dcb5a3dc/882d1050-e467-458c-aabe-cad74417742a"
-          (reference "C56") (unit 1)
+          (reference "C58") (unit 1)
         )
       )
@@
   )
   (symbol (lib_id "Commodore-2031:6522") (at 55.88 76.2 0) (unit 1)
-    (in_bom yes) (on_board yes) (dnp no) (fields_autoplaced)
-    (property "Reference" "UH3" (at 55.88 39.37 0)
-      (effects (font (size 1.27 1.27)))
-    )
-    (property "Value" "~" (at 55.88 55.88 0)
+    (in_bom yes) (on_board yes) (dnp no)
+    (property "Reference" "UH3" (at 55.88 36.83 0)
+      (effects (font (size 1.27 1.27)))
+    )
+    (property "Value" "6522" (at 55.88 39.37 0)
       (effects (font (size 1.27 1.27)))
     )
@@
   (symbol (lib_id "Device:C_Small") (at 191.77 123.19 0) (unit 1)
     (in_bom yes) (on_board yes) (dnp no) (fields_autoplaced)
-    (property "Reference" "C1" (at 194.31 122.5613 0)
+    (property "Reference" "C53" (at 194.31 122.5613 0)
       (effects (font (size 1.27 1.27)) (justify left))
     )
@@
       (project "Commodore-2031"
         (path "/4559151c-aecb-4a2a-972f-dcb7dcb5a3dc/882d1050-e467-458c-aabe-cad74417742a"
-          (reference "C1") (unit 1)
-        )
-      )
+          (reference "C53") (unit 1)
+        )
+      )

Commit message: Work towards ERC
- Add power flags
- Try to make sense of ground symbols
Connections:
- net GND renamed Earth
Changed lines of the file:
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@@
     )
   )
-  (symbol (lib_id "power:GND") (at 227.33 110.49 0) (unit 1)
+  (symbol (lib_id "power:Earth") (at 227.33 110.49 0) (unit 1)
     (in_bom yes) (on_board yes) (dnp no) (fields_autoplaced)
     (property "Reference" "#PWR033" (at 227.33 116.84 0)
@@
       (effects (font (size 1.27 1.27)) hide)
     )
-    (property "Datasheet" "" (at 227.33 110.49 0)
+    (property "Datasheet" "~" (at 227.33 110.49 0)
       (effects (font (size 1.27 1.27)) hide)
     )
@@
     )
   )
-  (symbol (lib_id "power:GND") (at 200.66 128.27 0) (unit 1)
+  (symbol (lib_id "power:Earth") (at 200.66 128.27 0) (unit 1)
     (in_bom yes) (on_board yes) (dnp no) (fields_autoplaced)
     (property "Reference" "#PWR034" (at 200.66 134.62 0)
@@
       (effects (font (size 1.27 1.27)) hide)
     )
-    (property "Datasheet" "" (at 200.66 128.27 0)
+    (property "Datasheet" "~" (at 200.66 128.27 0)
       (effects (font (size 1.27 1.27)) hide)
     )
@@
     )
   )
-  (symbol (lib_id "power:GND") (at 218.44 68.58 0) (unit 1)
+  (symbol (lib_id "power:Earth") (at 218.44 68.58 0) (unit 1)
     (in_bom yes) (on_board yes) (dnp no) (fields_autoplaced)
     (property "Reference" "#PWR029" (at 218.44 74.93 0)
@@
       (effects (font (size 1.27 1.27)) hide)
     )
-    (property "Datasheet" "" (at 218.44 68.58 0)
+    (property "Datasheet" "~" (at 218.44 68.58 0)
       (effects (font (size 1.27 1.27)) hide)
     )
@@
     )
   )
-  (symbol (lib_id "power:GND") (at 55.88 115.57 0) (unit 1)
+  (symbol (lib_id "power:Earth") (at 55.88 115.57 0) (unit 1)
     (in_bom yes) (on_board yes) (dnp no) (fields_autoplaced)
     (property "Reference" "#PWR023" (at 55.88 121.92 0)
@@
       (effects (font (size 1.27 1.27)) hide)
     )
-    (property "Datasheet" "" (at 55.88 115.57 0)
+    (property "Datasheet" "~" (at 55.88 115.57 0)
       (effects (font (size 1.27 1.27)) hide)
     )
@@
     )
   )
-  (symbol (lib_id "power:GND") (at 172.72 76.2 0) (unit 1)
+  (symbol (lib_id "power:Earth") (at 172.72 76.2 0) (unit 1)
     (in_bom yes) (on_board yes) (dnp no) (fields_autoplaced)
     (property "Reference" "#PWR044" (at 172.72 82.55 0)
@@
       (effects (font (size 1.27 1.27)) hide)
     )
-    (property "Datasheet" "" (at 172.72 76.2 0)
+    (property "Datasheet" "~" (at 172.72 76.2 0)
       (effects (font (size 1.27 1.27)) hide)
     )
@@
     )
   )
-  (symbol (lib_id "power:GND") (at 269.24 125.73 0) (unit 1)
+  (symbol (lib_id "power:Earth") (at 269.24 125.73 0) (unit 1)
     (in_bom yes) (on_board yes) (dnp no) (fields_autoplaced)
     (property "Reference" "#PWR036" (at 269.24 132.08 0)
@@
       (effects (font (size 1.27 1.27)) hide)
     )
-    (property "Datasheet" "" (at 269.24 125.73 0)
+    (property "Datasheet" "~" (at 269.24 125.73 0)
       (effects (font (size 1.27 1.27)) hide)
     )
@@
     )
   )
-  (symbol (lib_id "power:GND") (at 80.01 179.07 0) (unit 1)
+  (symbol (lib_id "power:Earth") (at 80.01 179.07 0) (unit 1)
     (in_bom yes) (on_board yes) (dnp no) (fields_autoplaced)
     (property "Reference" "#PWR027" (at 80.01 185.42 0)
@@
       (effects (font (size 1.27 1.27)) hide)
     )
-    (property "Datasheet" "" (at 80.01 179.07 0)
+    (property "Datasheet" "~" (at 80.01 179.07 0)
       (effects (font (size 1.27 1.27)) hide)
     )
@@
     )
   )
-  (symbol (lib_id "power:GND") (at 195.58 83.82 0) (unit 1)
+  (symbol (lib_id "power:Earth") (at 195.58 83.82 0) (unit 1)
     (in_bom yes) (on_board yes) (dnp no) (fields_autoplaced)
     (property "Reference" "#PWR032" (at 195.58 90.17 0)
@@
       (effects (font (size 1.27 1.27)) hide)
     )
-    (property "Datasheet" "" (at 195.58 83.82 0)
+    (property "Datasheet" "~" (at 195.58 83.82 0)
       (effects (font (size 1.27 1.27)) hide)
     )
@@
     )
   )
-  (symbol (lib_id "power:GND") (at 57.15 140.97 0) (unit 1)
+  (symbol (lib_id "power:Earth") (at 57.15 140.97 0) (unit 1)
     (in_bom yes) (on_board yes) (dnp no) (fields_autoplaced)
     (property "Reference" "#PWR024" (at 57.15 147.32 0)
@@
       (effects (font (size 1.27 1.27)) hide)
     )
-    (property "Datasheet" "" (at 57.15 140.97 0)
+    (property "Datasheet" "~" (at 57.15 140.97 0)
       (effects (font (size 1.27 1.27)) hide)
     )
@@
     )
   )
-  (symbol (lib_id "power:GND") (at 218.44 48.26 0) (unit 1)
+  (symbol (lib_id "power:Earth") (at 218.44 48.26 0) (unit 1)
     (in_bom yes) (on_board yes) (dnp no) (fields_autoplaced)
     (property "Reference" "#PWR028" (at 218.44 54.61 0)
@@
       (effects (font (size 1.27 1.27)) hide)
     )
-    (property "Datasheet" "" (at 218.44 48.26 0)
+    (property "Datasheet" "~" (at 218.44 48.26 0)
       (effects (font (size 1.27 1.27)) hide)
     )
@@
     )
   )
-  (symbol (lib_id "power:GND") (at 167.64 59.69 0) (unit 1)
+  (symbol (lib_id "power:Earth") (at 167.64 59.69 0) (unit 1)
     (in_bom yes) (on_board yes) (dnp no) (fields_autoplaced)
     (property "Reference" "#PWR030" (at 167.64 66.04 0)
@@
       (effects (font (size 1.27 1.27)) hide)
     )
-    (property "Datasheet" "" (at 167.64 59.69 0)
+    (property "Datasheet" "~" (at 167.64 59.69 0)
       (effects (font (size 1.27 1.27)) hide)
     )
@@
     )
   )
-  (symbol (lib_id "power:GND") (at 92.71 162.56 0) (unit 1)
+  (symbol (lib_id "power:Earth") (at 92.71 162.56 0) (unit 1)
     (in_bom yes) (on_board yes) (dnp no) (fields_autoplaced)
     (property "Reference" "#PWR026" (at 92.71 168.91 0)
@@
       (effects (font (size 1.27 1.27)) hide)
     )
-    (property "Datasheet" "" (at 92.71 162.56 0)
-      (effects (font (size 1.27 1.27)) hide)
-    )
+    (property "Datasheet" "~" (at 92.71 162.56 0)
+      (effects (font (size 1.27 1.27)) hide)
+    )

Commit message: Place capacitors and power units
Almost an error-free ERC!
Other:
- moved on the sheet: FB17
Changed lines of the file:
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@@
   (junction (at 209.55 58.42) (diameter 0) (color 0 0 0 0)
   )
+  (junction (at 274.32 125.73) (diameter 0) (color 0 0 0 0)
+  )
   (junction (at 227.33 109.22) (diameter 0) (color 0 0 0 0)
   )
@@
   )
   (junction (at 77.47 132.08) (diameter 0) (color 0 0 0 0)
+  )
+  (junction (at 185.42 73.66) (diameter 0) (color 0 0 0 0)
   )
   (junction (at 209.55 38.1) (diameter 0) (color 0 0 0 0)
@@
     (stroke (width 0) (type default))
   )
+  (wire (pts (xy 274.32 125.73) (xy 274.32 128.27))
+    (stroke (width 0) (type default))
+  )
   (wire (pts (xy 74.93 163.83) (xy 74.93 171.45))
     (stroke (width 0) (type default))
@@
     (stroke (width 0) (type default))
   )
+  (wire (pts (xy 274.32 125.73) (xy 276.86 125.73))
+    (stroke (width 0) (type default))
+  )
   (wire (pts (xy 92.71 153.67) (xy 92.71 156.21))
     (stroke (width 0) (type default))
@@
     (stroke (width 0) (type default))
   )
-  (wire (pts (xy 181.61 73.66) (xy 184.15 73.66))
+  (wire (pts (xy 181.61 73.66) (xy 185.42 73.66))
     (stroke (width 0) (type default))
   )
@@
     (stroke (width 0) (type default))
   )
+  (wire (pts (xy 185.42 72.39) (xy 185.42 73.66))
+    (stroke (width 0) (type default))
+  )
   (wire (pts (xy 38.1 53.34) (xy 43.18 53.34))
     (stroke (width 0) (type default))
@@
     (stroke (width 0) (type default))
   )
-  (wire (pts (xy 189.23 73.66) (xy 193.04 73.66))
-    (stroke (width 0) (type default))
-  )
-  (wire (pts (xy 269.24 124.46) (xy 269.24 125.73))
+  (wire (pts (xy 193.04 73.66) (xy 195.58 73.66))
+    (stroke (width 0) (type default))
+  )
+  (wire (pts (xy 269.24 124.46) (xy 269.24 128.27))
     (stroke (width 0) (type default))
   )
@@
   )
   (wire (pts (xy 218.44 99.06) (xy 218.44 102.87))
+    (stroke (width 0) (type default))
+  )
+  (wire (pts (xy 185.42 73.66) (xy 187.96 73.66))
     (stroke (width 0) (type default))
   )
@@
     (effects (font (size 2.54 2.54)) (justify left bottom))
   )
-  (text "pins 18-24 stacked (all ground)" (at 250.19 130.81 0)
+  (text "pins 18-24 stacked (all ground)" (at 250.19 133.35 0)
     (effects (font (size 1.27 1.27)) (justify left bottom))
   )
@@
     )
   )
-  (symbol (lib_id "Device:FerriteBead_Small") (at 186.69 73.66 90) (unit 1)
-    (in_bom yes) (on_board yes) (dnp no) (fields_autoplaced)
-    (property "Reference" "FB17" (at 186.6519 71.12 90)
-      (effects (font (size 1.27 1.27)))
-    )
-    (property "Value" "FerriteBead_Small" (at 186.6519 71.12 90)
-      (effects (font (size 1.27 1.27)) hide)
-    )
-    (property "Footprint" "" (at 186.69 75.438 90)
-      (effects (font (size 1.27 1.27)) hide)
-    )
-    (property "Datasheet" "~" (at 186.69 73.66 0)
+  (symbol (lib_id "Device:FerriteBead_Small") (at 190.5 73.66 90) (unit 1)
+    (in_bom yes) (on_board yes) (dnp no) (fields_autoplaced)
+    (property "Reference" "FB17" (at 190.4619 71.12 90)
+      (effects (font (size 1.27 1.27)))
+    )
+    (property "Value" "FerriteBead_Small" (at 190.4619 71.12 90)
+      (effects (font (size 1.27 1.27)) hide)
+    )
+    (property "Footprint" "" (at 190.5 75.438 90)
+      (effects (font (size 1.27 1.27)) hide)
+    )
+    (property "Datasheet" "~" (at 190.5 73.66 0)
       (effects (font (size 1.27 1.27)) hide)
     )
@@
         (path "/4559151c-aecb-4a2a-972f-dcb7dcb5a3dc/882d1050-e467-458c-aabe-cad74417742a"
           (reference "FB4") (unit 1)
+        )
+      )
+    )
+  )
+  (symbol (lib_id "power:PWR_FLAG") (at 276.86 125.73 270) (unit 1)
+    (in_bom yes) (on_board yes) (dnp no) (fields_autoplaced)
+    (property "Reference" "#FLG07" (at 278.765 125.73 0)
+      (effects (font (size 1.27 1.27)) hide)
+    )
+    (property "Value" "PWR_FLAG" (at 280.67 126.365 90)
+      (effects (font (size 1.27 1.27)) (justify left) hide)
+    )
+    (property "Footprint" "" (at 276.86 125.73 0)
+      (effects (font (size 1.27 1.27)) hide)
+    )
+    (property "Datasheet" "~" (at 276.86 125.73 0)
+      (effects (font (size 1.27 1.27)) hide)
+    )
+    (pin "1")
+    (instances
+      (project "Commodore-2031"
+        (path "/4559151c-aecb-4a2a-972f-dcb7dcb5a3dc/882d1050-e467-458c-aabe-cad74417742a"
+          (reference "#FLG07") (unit 1)
         )
       )
@@
     )
   )
-  (symbol (lib_id "power:GNDPWR") (at 274.32 125.73 0) (unit 1)
-    (in_bom yes) (on_board yes) (dnp no) (fields_autoplaced)
-    (property "Reference" "#PWR037" (at 274.32 130.81 0)
-      (effects (font (size 1.27 1.27)) hide)
-    )
-    (property "Value" "GNDPWR" (at 274.193 130.81 0)
-      (effects (font (size 1.27 1.27)) hide)
-    )
-    (property "Footprint" "" (at 274.32 127 0)
-      (effects (font (size 1.27 1.27)) hide)
-    )
-    (property "Datasheet" "" (at 274.32 127 0)
+  (symbol (lib_id "power:GNDPWR") (at 274.32 128.27 0) (unit 1)
+    (in_bom yes) (on_board yes) (dnp no) (fields_autoplaced)
+    (property "Reference" "#PWR037" (at 274.32 133.35 0)
+      (effects (font (size 1.27 1.27)) hide)
+    )
+    (property "Value" "GNDPWR" (at 274.193 133.35 0)
+      (effects (font (size 1.27 1.27)) hide)
+    )
+    (property "Footprint" "" (at 274.32 129.54 0)
+      (effects (font (size 1.27 1.27)) hide)
+    )
+    (property "Datasheet" "" (at 274.32 129.54 0)
       (effects (font (size 1.27 1.27)) hide)
     )
@@
     )
   )
-  (symbol (lib_id "power:Earth") (at 269.24 125.73 0) (unit 1)
-    (in_bom yes) (on_board yes) (dnp no) (fields_autoplaced)
-    (property "Reference" "#PWR036" (at 269.24 132.08 0)
-      (effects (font (size 1.27 1.27)) hide)
-    )
-    (property "Value" "GND" (at 269.24 130.81 0)
-      (effects (font (size 1.27 1.27)) hide)
-    )
-    (property "Footprint" "" (at 269.24 125.73 0)
-      (effects (font (size 1.27 1.27)) hide)
-    )
-    (property "Datasheet" "~" (at 269.24 125.73 0)
+  (symbol (lib_id "power:Earth") (at 269.24 128.27 0) (unit 1)
+    (in_bom yes) (on_board yes) (dnp no) (fields_autoplaced)
+    (property "Reference" "#PWR036" (at 269.24 134.62 0)
+      (effects (font (size 1.27 1.27)) hide)
+    )
+    (property "Value" "GND" (at 269.24 133.35 0)
+      (effects (font (size 1.27 1.27)) hide)
+    )
+    (property "Footprint" "" (at 269.24 128.27 0)
+      (effects (font (size 1.27 1.27)) hide)
+    )
+    (property "Datasheet" "~" (at 269.24 128.27 0)
       (effects (font (size 1.27 1.27)) hide)
     )
@@
     )
   )
-  (symbol (lib_id "power:+5V") (at 193.04 73.66 270) (unit 1)
-    (in_bom yes) (on_board yes) (dnp no) (fields_autoplaced)
-    (property "Reference" "#PWR031" (at 189.23 73.66 0)
-      (effects (font (size 1.27 1.27)) hide)
-    )
-    (property "Value" "+5V" (at 196.85 74.295 90)
-      (effects (font (size 1.27 1.27)) (justify left))
-    )
-    (property "Footprint" "" (at 193.04 73.66 0)
-      (effects (font (size 1.27 1.27)) hide)
-    )
-    (property "Datasheet" "" (at 193.04 73.66 0)
+  (symbol (lib_id "power:+5V") (at 195.58 73.66 270) (unit 1)
+    (in_bom yes) (on_board yes) (dnp no) (fields_autoplaced)
+    (property "Reference" "#PWR031" (at 191.77 73.66 0)
+      (effects (font (size 1.27 1.27)) hide)
+    )
+    (property "Value" "+5V" (at 199.39 74.295 90)
+      (effects (font (size 1.27 1.27)) (justify left))
+    )
+    (property "Footprint" "" (at 195.58 73.66 0)
+      (effects (font (size 1.27 1.27)) hide)
+    )
+    (property "Datasheet" "" (at 195.58 73.66 0)
       (effects (font (size 1.27 1.27)) hide)
     )
@@
         )
       )
+    )
+  )
+  (symbol (lib_id "power:PWR_FLAG") (at 185.42 72.39 0) (unit 1)
+    (in_bom yes) (on_board yes) (dnp no) (fields_autoplaced)
+    (property "Reference" "#FLG06" (at 185.42 70.485 0)
+      (effects (font (size 1.27 1.27)) hide)
+    )
+    (property "Value" "PWR_FLAG" (at 185.42 68.58 0)
+      (effects (font (size 1.27 1.27)) hide)
+    )
+    (property "Footprint" "" (at 185.42 72.39 0)
+      (effects (font (size 1.27 1.27)) hide)
+    )
+    (property "Datasheet" "~" (at 185.42 72.39 0)
+      (effects (font (size 1.27 1.27)) hide)
+    )
+    (pin "1")
+    (instances
+      (project "Commodore-2031"
+        (path "/4559151c-aecb-4a2a-972f-dcb7dcb5a3dc/882d1050-e467-458c-aabe-cad74417742a"
+          (reference "#FLG06") (unit 1)
+        )
+      )

Commit message: Resolve remaining ERC errors
... still lots of warnings tho.
Connections:
- no-connect marks 1 -> 3
Changed lines of the file:
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@@
     (comment 1 "Schematic 203138")
     (comment 2 "PCB Assembly 2031040")
+    (comment 4 "captured from original service manual by @rjhelms")
   )
   (junction (at 40.64 96.52) (diameter 0) (color 0 0 0 0)
@@
   )
   (no_connect (at 68.58 109.22))
+  (no_connect (at 69.85 91.44))
+  (no_connect (at 69.85 71.12))
   (bus_entry (at 74.93 53.34) (size 2.54 -2.54)
     (stroke (width 0) (type default))
