File: Commodore/2031/2031040/Commodore-2031/Sheet2-DriveSelectIEEE.kicad_sch (KiCad schematic)
At the start: 50 parts

Commit message: Verify schematic against parts list
A few discrepancies appear in original, these are noted in schematic.
Other:
- note added: "CR18 & CR19 are 1N270 in parts list"
Changed lines of the file:
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@@
-    (stroke (width 0) (type default))
-  )
-  (wire (pts (xy 209.55 125.73) (xy 209.55 127))
     (stroke (width 0) (type default))
   )
@@
     (stroke (width 0) (type default))
   )
-  (wire (pts (xy 200.66 127) (xy 209.55 127))
-    (stroke (width 0) (type default))
-  )
   (wire (pts (xy 252.73 93.98) (xy 264.16 93.98))
     (stroke (width 0) (type default))
@@
     (stroke (width 0) (type default))
   )
+  (text "CR18 & CR19 are 1N270 in parts list" (at 115.57 74.93 0)
+    (effects (font (size 1.27 1.27)) (justify left bottom))
+  )
   (text "DEVICE #\nSELECTION" (at 90.17 67.31 0)
